File: PIC/Dimmer/Dimmer.kicad_pcb (KiCad board)
At the start: 2 copper layers, 29 parts, among them J1 AC OUT, J2 AC IN, Q1 BC850, Q2 BC850, Q3 BC850, Q4 BT136-600, U1 PIC16F676, U2 74HC595, U3 D198K, U4 D198K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

Commit message: finish PCB
Parts:
- removed D1: LED, LED_SMD:LED_1206_3216Metric
- removed R7: 1K, Resistor_SMD:R_1206_3216Metric
- added C2: 105, Capacitor_THT:C_Axial_L5.1mm_D3.1mm_P12.50mm_Horizontal, F.Cu at (134.0, 25.9)
- added D4: D_Zener, Diode_THT:D_DO-34_SOD68_P7.62mm_Horizontal, F.Cu at (147.1, 26.4)
- added H1: MountingHole, MountingHole:MountingHole_2.5mm_Pad_Via, F.Cu at (175.8, 37.0)
- added H2: MountingHole, MountingHole:MountingHole_2.5mm_Pad_Via, F.Cu at (110.0, 37.0)
- added J3: Conn_01x05_Male, Connector_PinHeader_2.54mm:PinHeader_1x05_P2.54mm_Vertical, F.Cu at (228.6, 31.5)
- added J4: Conn_01x05_Male, Connector_PinHeader_2.54mm:PinHeader_1x05_P2.54mm_Vertical, F.Cu at (162.8, 31.5)
- added R12: 1M, Resistor_THT:R_Axial_DIN0204_L3.6mm_D1.6mm_P7.62mm_Horizontal, F.Cu at (130.8, 29.7)
- added R13: 10K, Resistor_THT:R_Axial_DIN0204_L3.6mm_D1.6mm_P7.62mm_Horizontal, F.Cu at (130.8, 32.5)
- Q1, Q2, Q3, R1, R10, R11, R2, R3, R4, R5, R6, R8, R9, U1, U2: moved to B.Cu
- RV1: footprint Potentiometer_THT:Potentiometer_Alps_RK163_Single_Horizontal -> Potentiometer_THT:Potentiometer_Bourns_3266Z_Horizontal
- moved R3 118.9 mm to (208.7, 40.0), turned to 180 degrees
- moved J2 112.2 mm to (109.7, 25.9)
- moved J1 107.7 mm to (109.7, 43.2)
- moved R5 92.5 mm to (208.7, 35.0), turned to 180 degrees
- moved R1 74.6 mm to (222.9, 33.8), turned to -90 degrees
- moved Q1 70.2 mm to (203.0, 40.4), turned to 90 degrees
- moved C1 67.1 mm to (153.9, 27.2), turned to 180 degrees
- moved R4 65.5 mm to (208.7, 37.5), turned to 180 degrees
- moved R8 65.4 mm to (154.2, 36.6), turned to 180 degrees
- moved Q3 57.0 mm to (203.1, 32.6), turned to 90 degrees
- moved Q2 49.6 mm to (203.0, 36.5), turned to 90 degrees
- moved U6 37.2 mm to (135.6, 42.4)
- moved RV1 34.5 mm to (223.4, 46.1), turned to 180 degrees
- moved D3 34.2 mm to (137.9, 31.5), turned to 90 degrees
- moved R2 32.7 mm to (223.4, 42.8), turned to 90 degrees
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Connections:
- C1 pad 2: GND -> Net-(C1-Pad2)
- D2 pad 4: Net-(D2-Pad4) -> Net-(C2-Pad2)
- D3 pad 3: GND -> Net-(C1-Pad2)
- D3 pad 4: Net-(D2-Pad4) -> Net-(C2-Pad1)
- J1 pad 1: Net-(D3-Pad2) -> Net-(J1-Pad1)
- J2 pad 1: Net-(D2-Pad4) -> Net-(C2-Pad2)
- J2 pad 2: Net-(D3-Pad2) -> Net-(J1-Pad1)
- Q4 pad 2: Net-(D2-Pad4) -> Net-(C2-Pad2)
- R10 pad 2: Net-(D3-Pad2) -> Net-(J1-Pad1)
- R11 pad 2: Net-(D2-Pad4) -> Net-(C2-Pad2)
- R6 pad 1: ZC -> Net-(C1-Pad1)
- R6 pad 2: VDD -> Net-(J4-Pad2)
- R8 pad 1: DIM -> Net-(J4-Pad3)
- R9 pad 2: Net-(D3-Pad2) -> Net-(J1-Pad1)
- U1 pad 5: SHCP -> DS
- U1 pad 6: DS -> SHCP
- U6 pad 4: GND -> Net-(C1-Pad2)
- U6 pad 5: ZC -> Net-(J4-Pad2)
- U7 pad 2: GND -> Net-(C1-Pad2)
Routing:
- net Net-(C1-Pad2): track 0.00 -> 72.2 mm
- net VDD: track 0.00 -> 71.1 mm, vias 0 -> 2
- net Net-(C2-Pad2): track 0.00 -> 64.9 mm, vias 0 -> 2
- net data5: track 0.00 -> 53.3 mm, vias 0 -> 3
- net data6: track 0.00 -> 52.9 mm, vias 0 -> 3
- net Net-(Q1-Pad3): track 0.00 -> 52.7 mm, vias 0 -> 3
- net data7: track 0.00 -> 50.9 mm, vias 0 -> 4
- net data4: track 0.00 -> 45.8 mm, vias 0 -> 3
- net STCP: track 0.00 -> 44.1 mm, vias 0 -> 2
- net data3: track 0.00 -> 42.5 mm, vias 0 -> 3
- net data1: track 0.00 -> 41.9 mm, vias 0 -> 3
- net SHCP: track 0.00 -> 41.8 mm, vias 0 -> 2
- net Net-(Q4-Pad3): track 0.00 -> 40.3 mm, vias 0 -> 2
- net data0: track 0.00 -> 39.3 mm, vias 0 -> 3
- net Net-(J4-Pad2): track 0.00 -> 38.4 mm
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- added copper zone on B.Cu, net GND
- added copper zone on F.Cu, net GND
Other:
- board outline added: 131.8 x 31 mm
