File: PIC/Dimmer/Dimmer.kicad_sch (KiCad schematic)
At the start: 29 parts

Commit message: add board file
Parts:
- C1: renamed from C?; footprint (none) -> Capacitor_THT:CP_Radial_D6.3mm_P2.50mm
- D1: renamed from D?; footprint (none) -> LED_SMD:LED_1206_3216Metric
- J1, J2: renamed from J?; footprint (none) -> TerminalBlock_Phoenix:TerminalBlock_Phoenix_MKDS-1,5-2_1x02_P5.00mm_Horizontal
- R1, R10, R11, R2, R3, R4, R5, R6, R7, R8, R9: renamed from R?; footprint (none) -> Resistor_SMD:R_1206_3216Metric
- RV1: renamed from RV?; footprint (none) -> Potentiometer_THT:Potentiometer_ACP_CA9-H2,5_Horizontal
- U7: renamed from U?; footprint (none) -> Package_DIP:DIP-6_W7.62mm
- gave numbers to parts that had none: 12

Commit message: finish PCB
Parts:
- removed D1: LED, LED_SMD:LED_1206_3216Metric, symbol Device:LED
- removed R7: 1K, Resistor_SMD:R_1206_3216Metric, symbol Device:R
- added C2: 105, Capacitor_THT:C_Axial_L5.1mm_D3.1mm_P12.50mm_Horizontal, symbol Device:C
- added D4: D_Zener, Diode_THT:D_DO-34_SOD68_P7.62mm_Horizontal, symbol Device:D_Zener
- added H1, H2: MountingHole, MountingHole:MountingHole_2.5mm_Pad_Via, symbol Mechanical:MountingHole
- added J3, J4: Conn_01x05_Male, Connector_PinHeader_2.54mm:PinHeader_1x05_P2.54mm_Vertical, symbol Connector:Conn_01x05_Male
- added R12: 1M, Resistor_THT:R_Axial_DIN0204_L3.6mm_D1.6mm_P7.62mm_Horizontal, symbol Device:R
- added R13: 10K, Resistor_THT:R_Axial_DIN0204_L3.6mm_D1.6mm_P7.62mm_Horizontal, symbol Device:R
- RV1: footprint Potentiometer_THT:Potentiometer_ACP_CA9-H2,5_Horizontal -> Potentiometer_THT:Potentiometer_Bourns_3266Z_Horizontal
Connections:
- net DIM: now also J3.3 (Pin_3); no longer R8.1
- net DS: now also U1.5 (RC5); no longer U1.6 (RC4)
- net GND: now also J3.4 (Pin_4), J3.5 (Pin_5); no longer C1.2, D3.3 (-), U6.4, U7.2
- net SHCP: now also U1.6 (RC4); no longer U1.5 (RC5)
- net VDD: now also J3.1 (Pin_1); no longer R6.2
- net ZC: now also J3.2 (Pin_2); no longer R6.1, U6.5
- net at J1.1 (Pin_1), J2.2 (Pin_2), R10.2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: now also R13.2; no longer D3.2
- net at C1.1, D3.1 (+): now also R6.1, D4.2 (A), J4.1 (Pin_1)
- net at D2.4, J2.1 (Pin_1), Q4.2 (A2)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: now also C2.2, R12.2; no longer D3.4
- new net: J4.2 (Pin_2), R6.2, U6.5
- new net: J4.3 (Pin_3), R8.1
- new net: C1.2, D3.3 (-), D4.1 (K), J4.4 (Pin_4), J4.5 (Pin_5), U6.4, U7.2
- new net: D3.2, R13.1
- new net: C2.1, D3.4, R12.1
Other:
- moved on the sheet: C1, D3, R6
